File: RFM69W.brd (EAGLE design)
At the start: 25.4 x 34.3 mm, 18 parts, among them U1 RFM69W, U2 MCP1701

Commit message: Updated README to confirm tested
Also filled in value on bypass cap.
Parts:
- C1: value (none) -> 0.1uF
Changed lines of the file:
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@@
 <attribute name="VALUE" x="2.794" y="11.303" size="0.4064" layer="27"/>
 </element>
-<element name="C1" library="SparkFun-Capacitors" package="0805" value="" x="1.27" y="6.35" smashed="yes" rot="R90">
+<element name="C1" library="SparkFun-Capacitors" package="0805" value="0.1uF" x="1.27" y="6.35" smashed="yes" rot="R90">
 <attribute name="NAME" x="2.9845" y="5.842" size="0.4064" layer="25" rot="R180"/>
 <attribute name="VALUE" x="2.667" y="5.334" size="0.4064" layer="27" rot="R90"/>
